File: v1/RampedFetCoil.kicad_pcb (KiCad board)
At the start: 2 copper layers, 76 x 228 mm, 113 parts, among them J1 FTSH-105-01-L-DV-K-P, J2 Conn_01x06, J3 703W-00_52, J4 Conn_01x01, J5 Conn_01x01, J6 Conn_01x01, J7 Conn_01x01, K1 G5Q-1A DC12, M1 Fan_CPU_4pin, Q10 Q_NMOS_GDS, Q5 T2N7002AK, Q6 T2N7002AK, Q7 Q_NMOS_GDS, Q8 Q_NMOS_GDS, Q9 Q_NMOS_GDS, T1 7492540200, U1 STM32G431KBTx, U10 SN74LV1T34DBV, U12 NCP1117-5.0_SOT223, U2 NCP1117-12_SOT223, U3 2ED2184S06F, U4 CSTNE8M00G550000R0, U5 NCP1117-3.3_SOT223, U6 MCP9700T-E/TT, U7 LNK306DG-TL, U8 2ED2184S06F, U9 IF D95-T

Commit message: sicswap
Parts:
- removed C15, C18: 0.1u, Capacitor_SMD:C_0805_2012Metric
- removed C19, C2: 2u2, Capacitor_SMD:C_0805_2012Metric
- removed Q10, Q8, Q9: Q_NMOS_GDS, Package_TO_SOT_THT:TO-247-3_Vertical
- removed R13, R14, R15, R9: 1.8R, Resistor_SMD:R_0805_2012Metric
- removed R30, R31: 2k, Resistor_SMD:R_0805_2012Metric
- removed U3, U8: 2ED2184S06F, Package_SO:SOIC-8_3.9x4.9mm_P1.27mm
- added C31: C, Capacitor_SMD:C_0805_2012Metric, F.Cu at (97.2, 72.2)
- added C32: C, Capacitor_SMD:C_0805_2012Metric, F.Cu at (97.0, 87.5)
- added C33: 0.1u, Capacitor_SMD:C_0805_2012Metric, F.Cu at (90.5, 87.6)
- added D15: US2MA, Diode_SMD:D_SMA, F.Cu at (96.0, 69.0)
- added Q1: C3M0120100K, Package_TO_SOT_THT:TO-247-4_Vertical, F.Cu at (104.5, 56.8)
- added Q2: C3M0120100K, Package_TO_SOT_THT:TO-247-4_Vertical, F.Cu at (104.5, 78.6)
- added Q3: C3M0120100K, Package_TO_SOT_THT:TO-247-4_Vertical, F.Cu at (53.1, 74.6)
- added Q4: C3M0120100K, Package_TO_SOT_THT:TO-247-4_Vertical, F.Cu at (53.1, 81.2)
- added R32: R, Resistor_SMD:R_0805_2012Metric, F.Cu at (93.5, 72.2)
- added R33: R, Resistor_SMD:R_0805_2012Metric, F.Cu at (91.0, 91.8)
- added R34: R, Resistor_SMD:R_0805_2012Metric, F.Cu at (93.0, 87.6)
- added R35: R, Resistor_SMD:R_0805_2012Metric, F.Cu at (99.5, 87.5)
- added R36: R, Resistor_SMD:R_0805_2012Metric, F.Cu at (100.5, 69.0)
- added U11: UCC21520DW, Package_SO:SOIC-16W_7.5x10.3mm_P1.27mm, F.Cu at (95.0, 79.0)
- Q7: value Q_NMOS_GDS -> T2N7002AK; footprint Package_TO_SOT_THT:TO-247-3_Vertical -> Package_TO_SOT_SMD:SOT-23
- moved Q7 37.4 mm to (94.2, 91.8)
- moved J7 2.00 mm to (90.2, 98.8)
Connections:
- Q7 pad 1: G_U1 -> GD_A
- Q7 pad 2: VBUS -> GND
- Q7 pad 3: SW1 -> Net-(Q7-D)
Routing:
- net (no net): track 0.00 -> 24.6 mm
- net Net-(Q7-D): track 0.00 -> 22.4 mm
- net K_U1: track 0.00 -> 20.8 mm
- net GND: track 651.9 -> 633.2 mm
- net SW1: track 18.3 -> 0.00 mm
- net Net-(U3-HO): track 16.8 -> 0.00 mm
- net Net-(U8-LO): track 15.6 -> 0.00 mm
- net GD_A: track 148.1 -> 160.8 mm, vias 2 -> 1
- net K_L1: track 0.00 -> 12.2 mm
- net +3V3: track 219.3 -> 228.2 mm
- net GD_DIS: track 358.2 -> 349.6 mm, vias 4 -> 3
- net Net-(U11-DT): track 0.00 -> 7.49 mm
- net Net-(U11-OUTA): track 0.00 -> 7.14 mm
- net Net-(D15-K): track 0.00 -> 6.24 mm
- net Net-(U8-HO): track 5.99 -> 0.00 mm
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