File: v1/RampedFetCoil.kicad_sch (KiCad schematic)
At the start: 113 parts, among them J1 FTSH-105-01-L-DV-K-P, J2 Conn_01x06, J3 703W-00_52, J4 Conn_01x01, J5 Conn_01x01, J6 Conn_01x01, J7 Conn_01x01, K1 G5Q-1A DC12, M1 Fan_CPU_4pin, Q10 Q_NMOS_GDS, Q5 T2N7002AK, Q6 T2N7002AK, Q7 Q_NMOS_GDS, Q8 Q_NMOS_GDS, Q9 Q_NMOS_GDS, T1 7492540200, U1 STM32G431KBTx, U10 SN74LV1T34DBV, U12 NCP1117-5.0_SOT223, U2 NCP1117-12_SOT223, U3 2ED2184S06F, U4 CSTNE8M00G550000R0, U5 NCP1117-3.3_SOT223, U6 MCP9700T-E/TT, U7 LNK306DG-TL, U8 2ED2184S06F, U9 IF D95-T

Commit message: sicswap
Parts:
- removed C15, C18: 0.1u, Capacitor_SMD:C_0805_2012Metric, symbol Device:C
- removed C19, C2: 2u2, Capacitor_SMD:C_0805_2012Metric, symbol Device:C
- removed Q10, Q7, Q8, Q9: Q_NMOS_GDS, Package_TO_SOT_THT:TO-247-3_Vertical, symbol Transistor_FET:Q_NMOS_GDS
- removed R13, R14, R15, R9: 1.8R, Resistor_SMD:R_0805_2012Metric, symbol Device:R
- removed R30, R31: 2k, Resistor_SMD:R_0805_2012Metric, symbol Device:R
- removed U8: 2ED2184S06F, Package_SO:SOIC-8_3.9x4.9mm_P1.27mm, symbol New_Library:2ED2184S06FXUMA1
- added C31, C32: C, Capacitor_SMD:C_0805_2012Metric, symbol Device:C
- added C33: 0.1u, Capacitor_SMD:C_0805_2012Metric, symbol Device:C
- added D15: US2MA, Diode_SMD:D_SMA, symbol Diode:US2MA
- added Q1, Q2, Q3, Q4: C3M0120100K, Package_TO_SOT_THT:TO-247-4_Vertical, symbol Transistor_FET:C3M0120100K
- added Q7: T2N7002AK, Package_TO_SOT_SMD:SOT-23, symbol Transistor_FET:T2N7002AK
- added R32, R33, R34, R35, R36: R, Resistor_SMD:R_0805_2012Metric, symbol Device:R
- added U11: UCC21520DW, Package_SO:SOIC-16W_7.5x10.3mm_P1.27mm, symbol Driver_FET:UCC21520DW
- U3: value 2ED2184S06F -> 2ED2184S06FXUMA1; footprint Package_SO:SOIC-8_3.9x4.9mm_P1.27mm -> 2ED2184S06FXUMA1:SOIC127P600X172-8N
Connections:
- net +15V: now also C32.1, R32.1, U11.11 (VDDB); no longer U3.5 (VCC)
- net +3V3: now also C33.2, R33.1, U11.3 (VCCI), U11.8 (VCCI)
- net GD_A: now also Q7.1 (G), U11.1 (INA); no longer U3.1 (IN)
- net GD_DIS: now also U11.5 (DIS); no longer U3.2 (~{SD})
- net GND: now also C33.1, Q2.2 (S), Q4.2 (S), Q7.2 (S), R34.1, U11.4 (GND); no longer U3.3 (COM)
- net G_L1: now also Q2.4 (G), R35.2
- net G_L2: now also Q4.4 (G)
- net G_U1: now also Q1.4 (G), R36.2
- net G_U2: now also Q3.4 (G)
- net SW1: now also Q1.2 (S), Q2.1 (D); no longer U3.6 (VS)
- net SW2: now also Q3.2 (S), Q4.1 (D)
- net VBUS: now also Q1.1 (D), Q3.1 (D)
- new net: R35.1, U11.10 (OUTB)
- new net: R36.1, U11.15 (OUTA)
- new net: C31.1, D15.1 (K), U11.16 (VDDA)
- new net: Q7.3 (D), R33.2, U11.2 (INB)
- new net: R34.2, U11.6 (DT)
- new net: D15.2 (A), R32.2
- new net K_L1: C32.2, Q2.3 (DS), U11.9 (VSSB)
- new net K_L2: Q4.3 (DS)
- new net K_U1: C31.2, Q1.3 (DS), U11.14 (VSSA)
- new net K_U2: Q3.3 (DS)
