File: v2/RampedFetCoil.kicad_pcb (KiCad board)
At the start: 2 copper layers, 94.5 x 228 mm, 151 parts, among them J1 FTSH-105-01-L-DV-K-P, J2 36503305, J3 703W-00_52, J4 Conn_01x01, J5 Conn_01x01, J6 Conn_01x01, J7 Conn_01x01, K2 G5Q-1, M1 Fan_CPU_4pin, Q1 C3M0120100K, Q2 C3M0120100K, Q3 C3M0120100K, Q4 C3M0120100K, Q5 T2N7002AK, Q6 T2N7002AK, Q7 T2N7002AK, T1 7492540200, U1 STM32G431KBTx, U11 UCC21520DW, U13 MGJ1D121505VMC-R7, U14 UCC21520DW, U15 MGJ1D121505VMC-R7, U16 MGJ1D121505VMC-R7, U2 74LVC1G14, U3 AP3928S-13, U4 CSTNE8M00G550000R0, U5 NCP1117-3.3_SOT223, U6 MCP9700T-E/TT, U7 74LVC1G14, U8 MGJ1D121505VMC-R7, U9 IF D95-T

Commit message: sicswap 2
Parts:
- added TP1: TestPoint, TestPoint:TestPoint_Pad_1.5x1.5mm, B.Cu at (85.8, 205.6)
- added TP2: TestPoint, TestPoint:TestPoint_Pad_1.5x1.5mm, B.Cu at (88.7, 205.6)
- added TP3: TestPoint, TestPoint:TestPoint_Pad_1.5x1.5mm, B.Cu at (88.7, 202.7)
- added TP4: TestPoint, TestPoint:TestPoint_Pad_1.5x1.5mm, B.Cu at (85.8, 202.8)
- moved R44 1.05 mm to (108.3, 219.2)
- moved R43 0.95 mm to (108.3, 221.2)
Connections:
- U1 pad 11: unconnected-(U1-PA6-Pad11) -> Net-(U1-PA6)
- U1 pad 12: unconnected-(U1-PA7-Pad12) -> Net-(U1-PA7)
- U1 pad 13: unconnected-(U1-PB0-Pad13) -> Net-(U1-PB0)
Routing:
- net Net-(U1-PB0): track 0.00 -> 10.3 mm, vias 0 -> 1
- net Net-(U1-PA6): track 0.00 -> 10.0 mm, vias 0 -> 1
- net Net-(U1-PA7): track 0.00 -> 7.73 mm, vias 0 -> 1
- net +3V3: track 460.2 -> 462.1 mm, vias 11 -> 12
- net +12V: track 509.3 -> 510.7 mm
- net GND: track 671.4 -> 670.5 mm
Other:
- board text added: "3V3"
- board text added: "PA6"
- board text added: "PA7"
- board text added: "PB0"

Commit message: unsure
Parts:
- R34, R38: value R -> 5k1
- R35, R36, R39, R40: value R -> 10R
Changed lines of the file:
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@@
 			)
 		)
-		(property "Value" "R"
+		(property "Value" "10R"
 			(at 0 1.65 0)
 			(layer "F.Fab")
@@
 			)
 		)
-		(property "Value" "R"
+		(property "Value" "10R"
 			(at 0 1.65 90)
 			(layer "F.Fab")
@@
 			)
 		)
-		(property "Value" "R"
+		(property "Value" "10R"
 			(at 0 1.65 90)
 			(layer "F.Fab")
@@
 			)
 		)
-		(property "Value" "R"
+		(property "Value" "5k1"
 			(at 0 1.65 90)
 			(layer "F.Fab")
@@
 			)
 		)
-		(property "Value" "R"
+		(property "Value" "10R"
 			(at 0 1.65 90)
 			(layer "F.Fab")
@@
 			)
 		)
-		(property "Value" "R"
+		(property "Value" "5k1"
 			(at 0 1.65 90)
 			(layer "F.Fab")
