File: interrupter/interrupter.kicad_pcb (KiCad board)
At the start: 2 copper layers, 79.2 x 61 mm, 47 parts, among them J1 Conn_01x02_Pin, J2 Conn_01x02_Pin, J3 Conn_01x02_Pin, J4 Conn_02x04_Top_Bottom, J5 USB4125-GF-A-0190, J6 Conn_01x03_Pin, J7 Conn_01x03_Pin, J8 Conn_01x03_Pin, Q1 T2N7002AK, U1 NCP1117-3.3_SOT223, U2 STM32C011F6Px, U3 IF-E96E, U4 MCP73831-2-OT, Y1 CSTNE24M0VH3C000R0

Commit message: unsure
Parts:
- removed J3: Conn_01x02_Pin, Connector_Molex:Molex_KK-254_AE-6410-02A_1x02_P2.54mm_Vertical
- removed J4: Conn_02x04_Top_Bottom, Connector_PinHeader_2.54mm:PinHeader_2x04_P2.54mm_Vertical
- removed J6, J7, J8: Conn_01x03_Pin, Connector_Molex:Molex_KK-254_AE-6410-03A_1x03_P2.54mm_Vertical
- added RV3: PTV09A-4020U-B103, Potentiometer_THT:Potentiometer_Bourns_PTV09A-1_Single_Vertical, F.Cu at (145.6, 80.8)
- added RV4: PTV09A-4020U-B103, Potentiometer_THT:Potentiometer_Bourns_PTV09A-1_Single_Vertical, F.Cu at (145.6, 95.1)
- added RV5: PTV09A-4020U-B103, Potentiometer_THT:Potentiometer_Bourns_PTV09A-1_Single_Vertical, F.Cu at (145.6, 109.5)
- added S1: 100SP1T1B4M2QE, digikey-footprints:Toggle_Switch_100SP1T1B4M2QE, F.Cu at (193.8, 83.0)
- added SW1: PS1024ALRED, Library:SW_PS1024ALRED, F.Cu at (166.1, 88.0)
- J2: value Conn_01x02_Pin -> Conn_ARM_SWD_TagConnect_TC2030; footprint Connector_Molex:Molex_KK-254_AE-6410-02A_1x02_P2.54mm_Vertical -> Connector:Tag-Connect_TC2030-IDC-FP_2x03_P1.27mm_Vertical
- RV1, RV2: value PTV09A-4020U-B103 -> 3386P-1-103LF; footprint Potentiometer_THT:Potentiometer_Bourns_PTV09A-1_Single_Vertical -> Potentiometer_THT:Potentiometer_Bourns_3386P_Vertical
- moved J2 74.1 mm to (176.6, 87.0)
- moved RV1 48.4 mm to (164.9, 79.2), turned to 0 degrees
- moved RV2 24.7 mm to (176.0, 79.2), turned to 0 degrees
Connections:
- J2 pad 1: Net-(J2-Pin_1) -> +3.3V
- J2 pad 2: +3.3V -> DIO
- R8 pad 2: Net-(J2-Pin_1) -> Net-(R8-Pad2)
- R9 pad 1: Net-(J2-Pin_1) -> Net-(R8-Pad2)
- U2 pad 10: RX2 -> unconnected-(U2-PA3-Pad10)
- U2 pad 9: TX2 -> unconnected-(U2-PA2-Pad9)
Routing:
- net unconnected-(U2-PA2-Pad9): track 0.00 -> 21.6 mm
- net TX2: track 21.6 -> 0.00 mm
- net unconnected-(U2-PA3-Pad10): track 0.00 -> 18.1 mm
- net RX2: track 18.1 -> 0.00 mm
- net Net-(R8-Pad2): track 0.00 -> 9.52 mm
- net Net-(J2-Pin_1): track 9.52 -> 0.00 mm
