File: interrupter/interrupter.kicad_sch (KiCad schematic)
At the start: 47 parts, among them J1 Conn_01x02_Pin, J2 Conn_01x02_Pin, J3 Conn_01x02_Pin, J4 Conn_02x04_Top_Bottom, J5 USB4125-GF-A-0190, J6 Conn_01x03_Pin, J7 Conn_01x03_Pin, J8 Conn_01x03_Pin, Q1 T2N7002AK, U1 NCP1117-3.3_SOT223, U2 STM32C011F6Px, U3 IF-E96E, U4 MCP73831-2-OT, Y1 CSTNE24M0VH3C000R0

Commit message: unsure
Parts:
- removed J2, J3: Conn_01x02_Pin, Connector_Molex:Molex_KK-254_AE-6410-02A_1x02_P2.54mm_Vertical, symbol Connector:Conn_01x02_Pin
- removed J4: Conn_02x04_Top_Bottom, Connector_PinHeader_2.54mm:PinHeader_2x04_P2.54mm_Vertical, symbol Connector_Generic:Conn_02x04_Top_Bottom
- removed J6, J7, J8: Conn_01x03_Pin, Connector_Molex:Molex_KK-254_AE-6410-03A_1x03_P2.54mm_Vertical, symbol Connector:Conn_01x03_Pin
- removed RV1, RV2: PTV09A-4020U-B103, Potentiometer_THT:Potentiometer_Bourns_PTV09A-1_Single_Vertical, symbol Device:R_Potentiometer_Trim
- added J2: Conn_ARM_SWD_TagConnect_TC2030, Connector:Tag-Connect_TC2030-IDC-FP_2x03_P1.27mm_Vertical, symbol Connector:Conn_ARM_SWD_TagConnect_TC2030
- added RV1, RV2: 3386P-1-103LF, Potentiometer_THT:Potentiometer_Bourns_3386P_Vertical, symbol Device:R_Potentiometer
- added RV3, RV4, RV5: PTV09A-4020U-B103, Potentiometer_THT:Potentiometer_Bourns_PTV09A-1_Single_Vertical, symbol Device:R_Potentiometer_Trim
- added S1: 100SP1T1B4M2QE, digikey-footprints:Toggle_Switch_100SP1T1B4M2QE, symbol dk_Toggle-Switches:100SP1T1B4M2QE
- added SW1: PS1024ALRED, Library:SW_PS1024ALRED, symbol Switch:SW_Push
Connections:
- net +3.3V: now also J2.1 (VCC), RV1.1, RV2.1, RV3.1, RV4.1, RV5.1, S1.2 (Com), SW1.1
- net CLK: now also J2.4 (SWCLK)
- net DIO: now also J2.2 (SWDIO)
- net E_BPS: now also RV4.2
- net E_OT: now also RV5.2
- net E_VMAX: now also RV3.2
- net GND: now also J2.5 (GND), RV1.3, RV2.3, RV3.3, RV4.3, RV5.3
- net I_DTC: now also RV2.2
- net I_OCD: now also RV1.2
- net NRST: now also J2.3 (~{RESET})
- net at R10.2, R11.1: now also S1.3
- net at R8.2, R9.1: now also SW1.2
- net RX2: no longer names the net of U2.10 (PA3)
- net TX2: no longer names the net of U2.9 (PA2)
Other:
- moved on the sheet: C8, C9
